File: MudderBoard/MudderBoard.kicad_sch (KiCad schematic)
At the start: 0 parts

Commit message: PP
Other:
- note added: "PENIS"
Changed lines of the file:
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@@
 		(company "Iceberg ASV")
+	)
+	(text "PENIS\n"
+		(exclude_from_sim no)
+		(at 49.784 36.83 0)
+		(effects
+			(font
+				(size 2.54 2.54)
+				(thickness 0.508)
+				(bold yes)
+			)
+		)
 	)
 	(sheet_instances
