File: MudderBoard/untitled.kicad_sch (KiCad schematic)
At the start: 8 parts, among them U1 LM51231QRGRRQ1

Commit message: softstart_Lidar
Parts:
- removed R2: 49.3k, RT0603DRE0749K3L:RESC1608X55N, symbol RT0603DRE0749K3L:RT0603DRE0749K3L
- added C5: GCM188R71C274KA37D, GCM188R71C274KA37D:CAPC1608X90N, symbol GCM188R71C274KA37D:GCM188R71C274KA37D
- added R2: 43m, RLP73M2BR043JTD:RESC3115X65N, symbol RLP73M2BR043JTD:RLP73M2BR043JTD
Connections:
- net GND: now also C5.2
- net VCC: now also R2.1
- net at U1.17 (SS): now also C5.1
- net at L1.1, U1.2 (CSN): now also R2.2
Other:
- moved on the sheet: R1, U1

Commit message: schematic_controller update
Parts:
- added C6: 4.7uF, TAJB_AVX, symbol TAJB475K035RNJ:TAJB475K035RNJ
- C5: value GCM188R71C274KA37D -> 2.7nF
Connections:
- net GND: now also C6.2
- net VCC: now also U1.12 (MODE), U1.8 (BIAS)
- net at U1.9 (VCC): now also C6.1
Other:
- moved on the sheet: C5, L1, R1, R2, U1
