File: MudderBoard/untitled.kicad_sch (KiCad schematic)
At the start: 10 parts, among them U1 LM51231QRGRRQ1

Commit message: ULVO Lidar
Parts:
- added R3: 74.1k, RN73R1JTTD7412B25:RESC1608X55N, symbol RN73R1JTTD7412B25:RN73R1JTTD7412B25
- added R4: 7.5k, RC0603N_YAG, symbol RC0603FR_077K5L:RC0603FR-077K5L
Connections:
- net GND: now also R4.2
- net VCC: now also R3.1
- net at U1.13 (UVLO_EN): now also R3.2, R4.1

Commit message: Block Diagram
Parts:
- added C7: CL21B474KAFNNNG, CAP_CL_21_SAM, symbol CL21B474KAFNNNG:CL21B474KAFNNNG
- added R5: 21k, RMCF0402FT21K0:RESC1005X35N, symbol RMCF0402FT21K0:RMCF0402FT21K0
- added R6: 14k, RC0402N_YAG, symbol RC0402FR-0714KL:RC0402FR-0714KL
Connections:
- net GND: now also C7.2, R6.2
- net at U1.16 (VREF_RANGE): now also C7.1, R5.1
- net at U1.18 (TRK): now also R5.2, R6.1
