File: MudderBoard/jetson.kicad_sch (KiCad schematic)
At the start: 0 parts

Commit message: added jetson circuit
Parts:
- added C60: 220uF, symbol Device:C_Polarized
- added C62: 100n, 0603, symbol Device:C
- added C63: 1n, 0603, symbol Device:C
- added C64: 18n, symbol Device:C
- added C65: 10p, 0603, symbol Device:C
- added C66: 82uF, symbol Device:C_Polarized
- added D8: STPS20M100SG-TR, D2PAK_STM, symbol STPS20M100SG_TR:STPS20M100SG-TR
- added L6: L, symbol Device:L
- added Q6: CSD16327Q3, Package_SON:VSON-8_3.3x3.3mm_P0.65mm_NexFET, symbol Transistor_FET:CSD16327Q3
- added R47: 3.09k, symbol Device:R
- added R53: 40K, symbol Device:R
- added R54: 1k, symbol Device:R
- added R55: 14k, symbol Device:R
- added R56: 100, symbol Device:R
- added R57: 8m, symbol Device:R
- added U9: LM3488QMM/NOPB, DGK8, symbol LM388MMNOPB:LM3488QMM_NOPB
Connections:
- new net: R56.1, U9.1 (ISEN)
- new net: C65.1, Q6.5 (D), R56.2, R57.1
- new net: C64.2, R47.1
- new net: C63.1, C64.1, U9.2 (COMP)
- new net: R54.2, R55.2, U9.3 (FB)
- new net: Q6.4 (G), U9.6 (DR)
- new net: R53.1, U9.7 (FA/SYNC/SD)
- new net: C66.1, D8.3, R55.1
- new net: D8.1, D8.2, L6.1, Q6.1 (S), Q6.2 (S), Q6.3 (S)
- new net +BATT: C60.1, C62.1, L6.2, U9.8 (VIN)
- new net GND: C60.2, C62.2, C63.2, C65.2, C66.2, R47.2, R53.2, R54.1, R57.2, U9.4 (AGND), U9.5 (PGND)
Other:
- note added: "REVIEW: NEED OUTPUT BARREL CONNECTOR"
- note added: "REVIEW: PLACEHOLDER INDUCTOR, NEED TO MAKE FOOTPRINT"
- note added: "REVIEW: REVIEW FOOTPRINT SIZES FOR CAPS AND RES MAKE SURE BOM MATCHES"
- note added: "REVIEW: should we seperate PGND and AGND?"

Commit message: added all footprints to Jetson circuit
Parts:
- removed C60: 220uF, symbol Device:C_Polarized
- removed C66: 82uF, symbol Device:C_Polarized
- added C10: 220u, Jetson_lib:U2-P_NCH, symbol UUD1H221MNL1GS:UUD1H221MNL1GS
- added C11: 220u, Jetson_lib:CAP_35SVPF82M, symbol 35SVPF82M:35SVPF82M
- C62, C63, C65: footprint 0603 -> Capacitor_SMD:C_0805_2012Metric
- C64: footprint (none) -> Capacitor_SMD:C_0402_1005Metric
- D8: footprint D2PAK_STM -> Jetson_lib:D2PAK_STM
- L6: value L -> 4.7u; footprint (none) -> Jetson_lib:PA2240
- R47, R54, R55, R56: footprint (none) -> Resistor_SMD:R_0402_1005Metric
- R53: value 40K -> 46.4k; footprint (none) -> Resistor_SMD:R_0402_1005Metric
- R57: footprint (none) -> Resistor_SMD:R_0603_1608Metric
- U9: footprint DGK8 -> Jetson_lib:DGK8
Connections:
- net +BATT: now also C10.1
- net GND: now also C10.2, C11.2
- net at D8.3, R55.1: now also C11.1
Other:
- note added: "Cbyp"
- note added: "Ccomp1"
- note added: "Ccomp2"
- note added: "Cfilt"
- note added: "Cin"
- note added: "Cout"
- note added: "REVIEW: REVIEW Rsense size"
- note added: "Rcomp"
- note added: "Rfb1"
- note added: "Rfb2"
- note added: "Rfilt"
- note added: "Rsense"
- note added: "Rsync"
- note removed: "REVIEW: PLACEHOLDER INDUCTOR, NEED TO MAKE FOOTPRINT"
- note removed: "REVIEW: REVIEW FOOTPRINT SIZES FOR CAPS AND RES MAKE SURE BOM MATCHES"
