File: MudderBoard/pwm-dc.kicad_sch (KiCad schematic)
At the start: 19 parts, among them K1 AZ2850-2A-12DE, Q2 NPN, U5 LM339, U6 UA741, U7 UA741

Commit message: PWM-DC prelim layout
Connections:
- net GND: now also C19.1; no longer C19.2
- net THRUST_SIG: now also C19.2; no longer C19.1
Other:
- moved on the sheet: C19
Changed lines of the file:
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@@
 	(symbol
 		(lib_id "Device:C")
-		(at 165.1 36.83 0)
+		(at 165.1 36.83 180)
 		(unit 1)
 		(exclude_from_sim no)
@@
 					(size 1.27 1.27)
 				)
-				(justify left)
+				(justify right)
 			)
 		)
@@
 					(size 1.27 1.27)
 				)
-				(justify left)
+				(justify right)
 			)
 		)
 		(property "Footprint" "PDC_Foot:CAPC2012X135N"
-			(at 166.0652 40.64 0)
+			(at 164.1348 33.02 0)
 			(effects
 				(font
